File: 6502 V1.3.kicad_pcb (KiCad board)
At the start: 2 copper layers, 45 parts, among them J1 Conn_02x32_Counter_Clockwise, J2 USB_C_Receptacle, SW1 SW_DIP_x04, SW3 SW_MEC_5E, U1 W65C02SxP, U2 W65C22SxP, U3 SST39SF040, U4 W65C51NxP, U5 CY62256-70PC, U6 ATF22V10B-15GM/883, U7 FT230XS, X1 ACO-1MHz-A, X2 ACO-1.8432MHz-A

Commit message: Designed board
Parts:
- removed the R1 at (65.4, 185.7)
- removed R11: 5100, Resistor_SMD:R_1206_3216Metric
- removed the R3 at (65.4, 192.3)
- removed the R4 at (65.4, 195.6)
- removed the R7 at (71.0, 185.7)
- removed the R8 at (71.0, 189.0)
- removed the R9 at (71.0, 192.3)
- removed SW3: SW_MEC_5E, Button_Switch_THT:SW_PUSH_6mm
- added REF**: MountingHole_3.2mm_M3_DIN965_Pad, MountingHole:MountingHole_3.2mm_M3_DIN965_Pad, F.Cu at (167.6, 25.4)
- added REF**: MountingHole_3.2mm_M3_DIN965_Pad, MountingHole:MountingHole_3.2mm_M3_DIN965_Pad, F.Cu at (25.4, 25.4)
- added REF**: MountingHole_3.2mm_M3_DIN965_Pad, MountingHole:MountingHole_3.2mm_M3_DIN965_Pad, F.Cu at (167.6, 91.4)
- added REF**: MountingHole_3.2mm_M3_DIN965_Pad, MountingHole:MountingHole_3.2mm_M3_DIN965_Pad, F.Cu at (25.4, 91.4)
- added RN1: 1000, Resistor_SMD:R_Array_Convex_4x1206, F.Cu at (135.3, 77.2)
- added RN2: R_Pack04, Resistor_SMD:R_Array_Convex_4x1206, F.Cu at (87.0, 26.4)
- added SW1: SW_Push, Button_Switch_SMD:SW_SPST_EVQPE1, F.Cu at (144.8, 25.4)
- D1: value LED -> PWR
- J1: value Conn_02x32_Counter_Clockwise -> Conn_02x32_Odd_Even; footprint Connector_PinHeader_2.54mm:PinHeader_2x32_P2.54mm_Vertical -> Connector_PinSocket_2.54mm:PinSocket_2x32_P2.54mm_Vertical
- J2: value USB_C_Receptacle -> USB_C_Receptacle_USB2.0_16P; footprint Connector_USB:USB_C_Receptacle_G-Switch_GT-USB-7010ASV -> Connector_USB:USB_C_Receptacle_GCT_USB4105-xx-A_16P_TopMnt_Horizontal
- JP3: footprint Connector_PinHeader_2.00mm:PinHeader_1x02_P2.00mm_Vertical -> Connector_PinHeader_2.54mm:PinHeader_1x02_P2.54mm_Vertical
- R2: value 1000 -> 5100
- moved D3 212.6 mm to (167.6, 55.9)
- moved D1 211.2 mm to (167.6, 50.8)
- moved D2 205.8 mm to (167.6, 61.0)
- moved R9 194.1 mm to (152.4, 25.4), turned to -90 degrees
- moved R4 188.2 mm to (158.6, 35.6)
- moved R2 185.9 mm to (162.6, 30.5), turned to 90 degrees
- moved R1 178.5 mm to (40.6, 25.4), turned to 180 degrees
- moved R3 175.6 mm to (162.6, 45.7), turned to -90 degrees
- moved JP1 169.1 mm to (127.4, 68.6)
- moved JP2 169.1 mm to (132.1, 68.6)
- moved C6 169.0 mm to (132.5, 25.4)
- moved JP3 168.8 mm to (136.4, 68.6)
- moved R8 166.6 mm to (158.6, 40.6)
- moved R7 162.0 mm to (161.1, 50.8)
- moved R5 160.5 mm to (161.1, 55.9)
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- renumbered C5 to C1, C1 to C10, C8 to C2, C6 to C3, C9 to C4, C7 to C5, C10 to C6, C4 to C7, C2 to C8, C3 to C9, R6 to R1, R10 to R3, R12 to R4, R15 to R5, R16 to R6, R14 to R7, R13 to R8, R5 to R9, SW1 to SW2, U6 to U1, U1 to U2, U2 to U3, U3 to U5, U7 to U6, U5 to U7, X2 to X1, X1 to X2
Connections:
- C10 pad 1: Net-(C1-Pad1) -> GND
- C10 pad 2: Net-(SW3-A) -> ~{RST}
- C8 pad 1: USBD- -> PUSBD-
- D1 pad 1: GND -> Net-(D1-K)
- D1 pad 2: Net-(D1-A) -> VCC
- J1 pad 1: ~{IRQ}_{PORT} -> A_{0}
- J1 pad 10: PB_{3} -> unconnected-(J1-Pin_10-Pad10)
- J1 pad 11: PB_{2} -> A_{5}
- J1 pad 12: PB_{1} -> unconnected-(J1-Pin_12-Pad12)
- J1 pad 13: PB_{0} -> A_{6}
- J1 pad 14: VCC -> unconnected-(J1-Pin_14-Pad14)
- J1 pad 15: GND -> A_{7}
- J1 pad 16: CA_{2} -> PA_{0}
- J1 pad 17: CA_{1} -> A_{8}
- J1 pad 18: PA_{7} -> PA_{1}
- J1 pad 19: PA_{6} -> A_{9}
- J1 pad 2: VCC -> unconnected-(J1-Pin_2-Pad2)
- J1 pad 20: PA_{5} -> PA_{2}
- J1 pad 21: PA_{4} -> A_{10}
- J1 pad 23: PA_{2} -> A_{11}
- J1 pad 24: PA_{1} -> PA_{4}
- J1 pad 25: PA_{0} -> A_{12}
- J1 pad 26: unconnected-(J1-Pin_26-Pad26) -> PA_{5}
- J1 pad 27: unconnected-(J1-Pin_27-Pad27) -> A_{13}
- J1 pad 28: unconnected-(J1-Pin_28-Pad28) -> PA_{6}
- J1 pad 29: unconnected-(J1-Pin_29-Pad29) -> A_{14}
- J1 pad 3: GND -> A_{1}
- J1 pad 30: unconnected-(J1-Pin_30-Pad30) -> PA_{7}
- J1 pad 31: unconnected-(J1-Pin_31-Pad31) -> A_{15}
- J1 pad 32: unconnected-(J1-Pin_32-Pad32) -> CA_{1}
- J1 pad 33: A_{0} -> D_{0}
- J1 pad 34: A_{1} -> CA_{2}
- J1 pad 35: A_{2} -> D_{1}
- J1 pad 36: A_{3} -> GND
- J1 pad 37: A_{4} -> D_{2}
- J1 pad 38: A_{5} -> VCC
- J1 pad 39: A_{6} -> D_{3}
- J1 pad 4: CB_{2} -> unconnected-(J1-Pin_4-Pad4)
- J1 pad 40: A_{7} -> PB_{0}
- J1 pad 41: A_{8} -> D_{4}
- J1 pad 42: A_{9} -> PB_{1}
- J1 pad 43: A_{10} -> D_{5}
- J1 pad 44: A_{11} -> PB_{2}
- J1 pad 45: A_{12} -> D_{6}
- J1 pad 46: A_{13} -> PB_{3}
- J1 pad 47: A_{14} -> D_{7}
- J1 pad 48: A_{15} -> PB_{4}
- J1 pad 49: D_{0} -> INH
- J1 pad 5: CB_{1} -> A_{2}
- J1 pad 50: D_{1} -> PB_{5}
- J1 pad 51: D_{2} -> ~{ROMOE}
- J1 pad 52: D_{3} -> PB_{6}
- J1 pad 53: D_{4} -> ~{RAMCS}
- J1 pad 54: D_{5} -> PB_{7}
- J1 pad 55: D_{6} -> ~{VIACS}
- J1 pad 56: D_{7} -> CB_{1}
- J1 pad 57: INH -> ~{ACIACS}
- J1 pad 58: ~{ROMOE} -> CB_{2}
- J1 pad 59: ~{RAMCS} -> CLK
- J1 pad 6: PB_{7} -> unconnected-(J1-Pin_6-Pad6)
- J1 pad 60: ~{VIACS} -> GND
- J1 pad 61: ~{ACIACS} -> GND
- J1 pad 62: CLK -> VCC
- J1 pad 63: GND -> VCC
- J1 pad 64: VCC -> ~{IRQ}_{PORT}
- J1 pad 7: PB_{6} -> A_{3}
- J1 pad 8: PB_{5} -> unconnected-(J1-Pin_8-Pad8)
- J1 pad 9: PB_{4} -> A_{4}
- R2 pad 1: BS_{1} -> Net-(J2-SBU1)
- R7 pad 1: VCC -> GND
- R7 pad 2: Net-(D1-A) -> Net-(D1-K)
- R9 pad 1: Net-(SW3-A) -> ~{RST}
Other:
- board outline added: 152.4 x 76.2 mm

Commit message: More routing
Parts:
- moved SW1 0.52 mm to (71.1, 31.0), turned to -90 degrees
- renumbered C9 to C10, C4 to C2, C5 to C3, C3 to C4, C2 to C5, C8 to C7, C10 to C8, C7 to C9, D2 to D1, D1 to D2, J2 to J1, J1 to J2, JP2 to JP1, JP1 to JP2, R4 to R2, R2 to R3, R9 to R4, R8 to R7, R7 to R8, R3 to R9, RN2 to RN1, RN1 to RN2, SW2 to SW1, SW1 to SW2, U2 to U1, U3 to U2, U4 to U3, U7 to U4, U1 to U5, U5 to U7, X2 to X1, X1 to X2
Routing:
- net ~{IRQ}_{CPU}: track 0.00 -> 151.6 mm, vias 0 -> 1
- net CA_{2}: track 0.00 -> 135.1 mm, vias 0 -> 2
- net CA_{1}: track 0.00 -> 129.3 mm, vias 0 -> 3
- net ~{VIACS}: track 0.00 -> 128.6 mm, vias 0 -> 3
- net A_{9}: track 0.00 -> 99.8 mm, vias 0 -> 2
- net A_{11}: track 0.00 -> 94.1 mm
- net A_{7}: track 0.00 -> 93.6 mm, vias 0 -> 2
- net A_{8}: track 0.00 -> 92.6 mm, vias 0 -> 2
- net A_{5}: track 0.00 -> 92.0 mm, vias 0 -> 1
- net A_{4}: track 0.00 -> 91.8 mm, vias 0 -> 1
- net A_{6}: track 0.00 -> 91.6 mm, vias 0 -> 2
- net CB_{2}: track 0.00 -> 87.1 mm, vias 0 -> 1
- net PB_{1}: track 0.00 -> 87.0 mm, vias 0 -> 1
- net CB_{1}: track 0.00 -> 86.7 mm, vias 0 -> 1
- net PB_{7}: track 0.00 -> 86.7 mm, vias 0 -> 1
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