File: 6502 V1.3.kicad_pcb (KiCad board)
At the start: 2 copper layers, 152.4 x 76.2 mm, 44 parts, among them J1 USB_C_Receptacle_USB2.0_16P, J2 Conn_02x32_Odd_Even, SW1 SW_DIP_x04, SW2 SW_Push, U1 W65C02SxP, U2 W65C22SxP, U3 W65C51NxP, U4 CY62256-70PC, U5 ATF22V10B-15GM/883, U6 FT230XS, U7 SST39SF040, X1 ACO-1MHz-A, X2 ACO-1.8432MHz-A

Commit message: Fixed round traces
Routing:
- net GND: track 432.7 -> 448.4 mm, vias 22 -> 24
- net A_{5}: track 220.0 -> 226.2 mm
- net VCC: track 570.3 -> 575.9 mm
- net A_{7}: track 217.2 -> 221.2 mm
- net A_{6}: track 216.2 -> 219.7 mm
- net ~{IRQ}_{ACIA}: track 114.5 -> 117.3 mm
- net R/~{W}: track 182.9 -> 185.4 mm
- net CLK: track 312.0 -> 314.2 mm
- net A_{11}: track 251.1 -> 248.9 mm
- net ~{IRQ}_{CPU}: track 164.7 -> 166.8 mm
- net A_{1}: track 182.8 -> 184.4 mm
- net A_{12}: track 231.8 -> 233.3 mm
- net D_{3}: track 148.1 -> 149.6 mm
- net ~{IRQ}_{VIA}: track 154.4 -> 155.7 mm
- net D_{4}: track 161.3 -> 162.6 mm
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
Commit message: Finished tracing, corrected INH pull resistor
Parts:
- added R10: 1000, Resistor_SMD:R_1206_3216Metric, F.Cu at (113.3, 76.2)
- moved JP1 8.92 mm to (127.5, 68.6)
- moved JP3 4.65 mm to (132.1, 68.6)
- moved JP2 4.32 mm to (136.4, 68.6)
- renumbered C8 to C7, C7 to C8, R4 to R2, R2 to R3, R3 to R4, R6 to R5, R5 to R6, R9 to R7, R7 to R9
Connections:
- JP1 pad 1: ~{IRQ}_{PORT} -> ~{IRQ}_{VIA}
- JP1 pad 2: Net-(JP3-B) -> Net-(JP1-B)
- JP2 pad 1: ~{IRQ}_{ACIA} -> ~{IRQ}_{PORT}
- JP2 pad 2: Net-(JP2-B) -> Net-(JP3-B)
- JP3 pad 1: ~{IRQ}_{VIA} -> ~{IRQ}_{ACIA}
- JP3 pad 2: Net-(JP1-B) -> Net-(JP2-B)
Routing:
- net INH: track 51.8 -> 63.9 mm
- net GND: track 448.4 -> 451.1 mm
