File: Deadend.kicad_pcb (KiCad board)
At the start: 2 copper layers, 152.4 x 76.2 mm, 44 parts, among them J1 Conn_02x32_Odd_Even, J2 USB_C_Receptacle_USB2.0_16P, SW1 SW_Push, SW2 SW_DIP_x04, U1 ATF22V10B-15GM/883, U2 W65C02SxP, U3 W65C22SxP, U4 W65C51NxP, U5 SST39SF040, U6 FT230XS, U7 CY62256-70PC, X1 ACO-1.8432MHz-A, X2 ACO-1MHz-A

Commit message: More tracing1
Parts:
- moved J2 10.5 mm to (58.4, 86.4)
- renumbered C9 to C10, C4 to C2, C5 to C3, C3 to C4, C2 to C5, C8 to C7, C10 to C8, C7 to C9, D2 to D1, D1 to D2, J2 to J1, J1 to J2, JP2 to JP1, JP1 to JP2, R4 to R2, R2 to R3, R9 to R4, R8 to R7, R7 to R8, R3 to R9, RN2 to RN1, RN1 to RN2, SW2 to SW1, SW1 to SW2, U2 to U1, U3 to U2, U4 to U3, U7 to U4, U1 to U5, U5 to U7, X2 to X1, X1 to X2
Routing:
- net A_{8}: track 0.00 -> 251.2 mm, vias 0 -> 2
- net A_{11}: track 0.00 -> 247.9 mm, vias 0 -> 2
- net A_{9}: track 0.00 -> 247.7 mm, vias 0 -> 2
- net A_{10}: track 0.00 -> 240.3 mm, vias 0 -> 3
- net A_{14}: track 0.00 -> 235.4 mm, vias 0 -> 3
- net A_{12}: track 0.00 -> 232.3 mm, vias 0 -> 1
- net CLK: track 0.00 -> 228.2 mm, vias 0 -> 1
- net A_{15}: track 0.00 -> 226.9 mm, vias 0 -> 1
- net A_{13}: track 0.00 -> 223.7 mm, vias 0 -> 3
- net A_{7}: track 0.00 -> 219.8 mm, vias 0 -> 2
- net A_{6}: track 0.00 -> 218.4 mm, vias 0 -> 3
- net A_{5}: track 0.00 -> 218.3 mm, vias 0 -> 4
- net A_{4}: track 0.00 -> 212.3 mm, vias 0 -> 2
- net D_{7}: track 0.00 -> 181.7 mm, vias 0 -> 2
- net D_{6}: track 0.00 -> 180.0 mm, vias 0 -> 2
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