File: test.kicad_pcb (KiCad board)
At the start: 2 copper layers, 152.4 x 76.2 mm, 44 parts, among them J1 USB_C_Receptacle_USB2.0_16P, J2 Conn_02x32_Odd_Even, SW1 SW_DIP_x04, SW2 SW_Push, U1 W65C02SxP, U2 W65C22SxP, U3 W65C51NxP, U4 CY62256-70PC, U5 ATF22V10B-15GM/883, U6 FT230XS, U7 SST39SF040, X1 ACO-1MHz-A, X2 ACO-1.8432MHz-A

Commit message: Finished routing
Parts:
- moved RN1 2.58 mm to (132.7, 77.7)
- turned R4 to 180 degrees
- turned R8 to 180 degrees
- renumbered C8 to C10, C5 to C2, C4 to C3, C2 to C4, C3 to C5, C9 to C7, C7 to C8, C10 to C9, D2 to D1, D1 to D2, J2 to J1, J1 to J2, JP2 to JP1, JP1 to JP2, R3 to R2, R9 to R3, R2 to R4, R8 to R7, R7 to R8, R4 to R9, RN2 to RN1, RN1 to RN2, SW2 to SW1, SW1 to SW2, U5 to U1, U1 to U2, U2 to U3, U3 to U4, U7 to U5, U4 to U7, X2 to X1, X1 to X2
Connections:
- J1 pad 2: unconnected-(J1-Pin_2-Pad2) -> R/~{W}
Routing:
- net A_{8}: track 251.2 -> 0.00 mm, vias 2 -> 0
- net A_{11}: track 247.9 -> 0.00 mm, vias 2 -> 0
- net A_{9}: track 247.7 -> 0.00 mm, vias 2 -> 0
- net A_{10}: track 240.3 -> 0.00 mm, vias 3 -> 0
- net A_{14}: track 235.4 -> 0.00 mm, vias 3 -> 0
- net A_{12}: track 232.3 -> 0.00 mm, vias 1 -> 0
- net CLK: track 228.2 -> 0.00 mm, vias 1 -> 0
- net A_{15}: track 226.9 -> 0.00 mm, vias 1 -> 0
- net A_{13}: track 223.7 -> 0.00 mm, vias 3 -> 0
- net A_{7}: track 219.8 -> 0.00 mm, vias 2 -> 0
- net A_{6}: track 218.4 -> 0.00 mm, vias 3 -> 0
- net A_{5}: track 218.3 -> 0.00 mm, vias 4 -> 0
- net A_{4}: track 212.3 -> 0.00 mm, vias 2 -> 0
- net D_{7}: track 181.7 -> 0.00 mm, vias 2 -> 0
- net D_{6}: track 180.0 -> 0.00 mm, vias 2 -> 0
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