File: 6502 V1.3-rounded.kicad_pcb (KiCad board)
At the start: 2 copper layers, 152.4 x 76.2 mm, 44 parts, among them J1 USB_C_Receptacle_USB2.0_16P, J2 Conn_02x32_Odd_Even, SW1 SW_DIP_x04, SW2 SW_Push, U1 W65C02SxP, U2 W65C22SxP, U3 W65C51NxP, U4 CY62256-70PC, U5 ATF22V10B-15GM/883, U6 FT230XS, U7 SST39SF040, X1 ACO-1MHz-A, X2 ACO-1.8432MHz-A

Commit message: Finished routing
Routing:
- net A_{10}: track 244.5 -> 245.1 mm
Changed lines of the file:
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@@
   (via (at 83.058 29.718) (size 0.8) (drill 0.4) (layers "F.Cu" "B.Cu") (net 40))
   (via (at 78.74 73.66) (size 0.8) (drill 0.4) (layers "F.Cu" "B.Cu") (net 40))
+  (segment (start 78.486 66.802) (end 78.486 81.026) (width 0.25) (layer "B.Cu") (net 40))
+  (segment (start 81.275 64.77) (end 80.518 64.77) (width 0.25) (layer "B.Cu") (net 40))
+  (segment (start 80.518 64.77) (end 78.486 66.802) (width 0.25) (layer "B.Cu") (net 40))
   (segment (start 83.75 40.692812) (end 83.058 40.000812) (width 0.25) (layer "B.Cu") (net 40))
-  (segment (start 78.74 67.305) (end 78.74 81.28) (width 0.25) (layer "B.Cu") (net 40))
   (segment (start 83.058 62.6) (end 83.058 58.543396) (width 0.25) (layer "B.Cu") (net 40))
-  (segment (start 81.275 64.77) (end 78.74 67.305) (width 0.25) (layer "B.Cu") (net 40))
-  (segment (start 78.74 81.28) (end 83.82 86.36) (width 0.25) (layer "B.Cu") (net 40))
   (segment (start 83.058 40.000812) (end 83.058 29.718) (width 0.25) (layer "B.Cu") (net 40))
   (segment (start 83.058 58.543396) (end 83.75 57.851396) (width 0.25) (layer "B.Cu") (net 40))
   (segment (start 83.75 57.851396) (end 83.75 40.692812) (width 0.25) (layer "B.Cu") (net 40))
+  (segment (start 78.486 81.026) (end 83.82 86.36) (width 0.25) (layer "B.Cu") (net 40))
   (segment (start 83.958 63.5) (end 83.058 62.6) (width 0.25) (layer "B.Cu") (net 40))
   (segment (start 83.209 26.187396) (end 83.209 27.871808) (width 0.25) (layer "F.Cu") (net 41))

Commit message: Fixed round traces
Routing:
- net GND: track 432.7 -> 441.2 mm, vias 22 -> 24
- net A_{11}: track 251.1 -> 244.5 mm
- net A_{9}: track 251.6 -> 246.3 mm
- net A_{8}: track 255.3 -> 251.4 mm
- net A_{10}: track 245.1 -> 241.4 mm
- net VCC: track 570.3 -> 566.9 mm
- net A_{2}: track 172.5 -> 169.2 mm
- net A_{13}: track 223.5 -> 220.3 mm
- net A_{0}: track 171.7 -> 168.6 mm
- net A_{4}: track 211.7 -> 208.8 mm
- net A_{3}: track 173.7 -> 171.0 mm
- net D_{6}: track 179.9 -> 177.2 mm
- net A_{12}: track 231.8 -> 229.1 mm
- net D_{5}: track 170.5 -> 167.8 mm
- net A_{5}: track 220.0 -> 222.4 mm
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
Commit message: Finished tracing, corrected INH pull resistor
Parts:
- added G***: LOGO, delorean:unicorn, F.Cu at (147.8, 55.1)
- added R10: 1000, Resistor_SMD:R_1206_3216Metric, F.Cu at (113.3, 76.2)
- moved JP3 0.08 mm to (127.5, 68.6)
- renumbered C9 to C10, C8 to C7, C7 to C8, C10 to C9, D2 to D1, D1 to D2, R4 to R2, R2 to R3, R3 to R4, R7 to R5, R5 to R7, R9 to R8, R8 to R9
Routing:
- net INH: track 50.8 -> 62.9 mm
- net GND: track 441.2 -> 443.9 mm
Other:
- board text added: "22V10"
- board text added: "39SF040"
- board text added: "4 MHz CLK"
- board text added: "6502 SBC V1.3 Ethan Thummel 1/22/24"
- board text added: "6551"
- board text added: "65C02"
- board text added: "65C22"
- board text added: "A_{0}"
- board text added: "A_{10}"
- board text added: "A_{11}"
- board text added: "A_{12}"
- board text added: "A_{13}"
- board text added: "A_{14}"
- board text added: "A_{15}"
- board text added: "A_{1}"
- board text added: "A_{2}"
- board text added: "A_{3}"
- board text added: "A_{4}"
- board text added: "A_{5}"
- board text added: "A_{6}"
- board text added: "A_{7}"
- board text added: "A_{8}"
- board text added: "A_{9}"
- board text added: "BANK SELECT"
- board text added: "CA_{1}"
- board text added: "CA_{2}"
- board text added: "CB_{1}"
- board text added: "CB_{2}"
- board text added: "CLK"
- board text added: "D_{0}"
- board text added: "D_{1}"
- board text added: "D_{2}"
- board text added: "D_{3}"
- board text added: "D_{4}"
- board text added: "D_{5}"
- board text added: "D_{6}"
- board text added: "D_{7}"
- board text added: "GND"
- board text added: "HM62256B"
- board text added: "INH"
- board text added: "PA_{0}"
- board text added: "PA_{1}"
- board text added: "PA_{2}"
- board text added: "PA_{3}"
- board text added: "PA_{4}"
- board text added: "PA_{5}"
- board text added: "PA_{6}"
- board text added: "PA_{7}"
- board text added: "PB_{0}"
- board text added: "PB_{1}"
- board text added: "PB_{2}"
- board text added: "PB_{3}"
- board text added: "PB_{4}"
- board text added: "PB_{5}"
- board text added: "PB_{6}"
- board text added: "PB_{7}"
- board text added: "R/~{W}"
- board text added: "RST"
- board text added: "UART CLK"
- board text added: "VCC"
- board text added: "~{ACIACS}"
- board text added: "~{IRQ}"
- board text added: "~{IRQ}_{ACIA}"
- board text added: "~{IRQ}_{PORT}"
- board text added: "~{IRQ}_{VIA}"
- board text added: "~{RAMCS}"
- board text added: "~{ROMOE}"
- board text added: "~{VIACS}"
- board text added: "コンピューター！"
