File: 6502 V1.3.kicad_sch (KiCad schematic)
At the start: 45 parts, among them J1 Conn_02x32_Counter_Clockwise, J2 USB_C_Receptacle, SW1 SW_DIP_x04, SW3 SW_MEC_5E, U1 W65C02SxP, U2 W65C22SxP, U3 SST39SF040, U4 W65C51NxP, U5 CY62256-70PC, U6 ATF22V10B-15GM/883, U7 FT230XS, X1 ACO-1MHz-A, X2 ACO-1.8432MHz-A

Commit message: Designed board
Parts:
- removed J1: Conn_02x32_Counter_Clockwise, Connector_PinHeader_2.54mm:PinHeader_2x32_P2.54mm_Vertical, symbol Connector_Generic:Conn_02x32_Counter_Clockwise
- removed J2: USB_C_Receptacle, Connector_USB:USB_C_Receptacle_G-Switch_GT-USB-7010ASV, symbol Connector:USB_C_Receptacle
- removed R1, R3, R4, R7, R8, R9: 1000, Resistor_SMD:R_1206_3216Metric, symbol Device:R
- removed R11: 5100, Resistor_SMD:R_1206_3216Metric, symbol Device:R
- removed SW3: SW_MEC_5E, Button_Switch_THT:SW_PUSH_6mm, symbol Switch:SW_MEC_5E
- added J1: Conn_02x32_Odd_Even, Connector_PinSocket_2.54mm:PinSocket_2x32_P2.54mm_Vertical, symbol Connector_Generic:Conn_02x32_Odd_Even
- added J2: USB_C_Receptacle_USB2.0_16P, Connector_USB:USB_C_Receptacle_GCT_USB4105-xx-A_16P_TopMnt_Horizontal, symbol Connector:USB_C_Receptacle_USB2.0_16P
- added RN1: 1000, Resistor_SMD:R_Array_Convex_4x1206, symbol Device:R_Pack04
- added RN2: R_Pack04, Resistor_SMD:R_Array_Convex_4x1206, symbol Device:R_Pack04
- added SW1: SW_Push, Button_Switch_SMD:SW_SPST_EVQPE1, symbol Switch:SW_Push
- D1: value LED -> PWR
- JP3: footprint Connector_PinHeader_2.00mm:PinHeader_1x02_P2.00mm_Vertical -> Connector_PinHeader_2.54mm:PinHeader_1x02_P2.54mm_Vertical
- R2: value 1000 -> 5100
- renumbered C5 to C1, C1 to C10, C8 to C2, C6 to C3, C9 to C4, C7 to C5, C10 to C6, C4 to C7, C2 to C8, C3 to C9, R6 to R1, R10 to R3, R12 to R4, R15 to R5, R16 to R6, R14 to R7, R13 to R8, R5 to R9, SW1 to SW2, U6 to U1, U1 to U2, U2 to U3, U3 to U5, U7 to U6, U5 to U7, X2 to X1, X1 to X2
Connections:
- net A_{0}: now also J1.1 (Pin_1)
- net A_{10}: now also J1.21 (Pin_21)
- net A_{11}: now also J1.23 (Pin_23)
- net A_{12}: now also J1.25 (Pin_25)
- net A_{13}: now also J1.27 (Pin_27)
- net A_{14}: now also J1.29 (Pin_29)
- net A_{15}: now also J1.31 (Pin_31)
- net A_{1}: now also J1.3 (Pin_3)
- net A_{2}: now also J1.5 (Pin_5)
- net A_{3}: now also J1.7 (Pin_7)
- net A_{4}: now also J1.9 (Pin_9)
- net A_{5}: now also J1.11 (Pin_11)
- net A_{6}: now also J1.13 (Pin_13)
- net A_{7}: now also J1.15 (Pin_15)
- net A_{8}: now also J1.17 (Pin_17)
- net A_{9}: now also J1.19 (Pin_19)
- net BS_{0}: now also RN2.8 (R1.2)
- net BS_{1}: now also RN2.7 (R2.2); no longer R2.1
- net BS_{2}: now also RN2.6 (R3.2)
- net BS_{3}: now also RN2.5 (R4.2)
- net CA_{1}: now also J1.32 (Pin_32)
- net CA_{2}: now also J1.34 (Pin_34)
- net CB_{1}: now also J1.56 (Pin_56)
- net CB_{2}: now also J1.58 (Pin_58)
- net CLK: now also J1.59 (Pin_59)
- net D_{0}: now also J1.33 (Pin_33)
- net D_{1}: now also J1.35 (Pin_35)
- net D_{2}: now also J1.37 (Pin_37)
- net D_{3}: now also J1.39 (Pin_39)
- net D_{4}: now also J1.41 (Pin_41)
- net D_{5}: now also J1.43 (Pin_43)
- net D_{6}: now also J1.45 (Pin_45)
- net D_{7}: now also J1.47 (Pin_47)
- net GND: now also C10.1, R7.1, J1.36 (Pin_36), J1.60 (Pin_60), J1.61 (Pin_61), J2.A1 (GND), J2.A12 (GND), J2.B1 (GND), J2.B12 (GND), J2.S1 (SHIELD), RN2.1 (R1.1), RN2.2 (R2.1), RN2.3 (R3.1), RN2.4 (R4.1), SW1.1; no longer D1.1 (K)
- net INH: now also J1.49 (Pin_49)
- net PA_{0}: now also J1.16 (Pin_16)
- net PA_{1}: now also J1.18 (Pin_18)
- net PA_{2}: now also J1.20 (Pin_20)
- net PA_{3}: now also J1.22 (Pin_22)
- net PA_{4}: now also J1.24 (Pin_24)
- net PA_{5}: now also J1.26 (Pin_26)
- net PA_{6}: now also J1.28 (Pin_28)
- net PA_{7}: now also J1.30 (Pin_30)
- net PB_{0}: now also J1.40 (Pin_40)
- net PB_{1}: now also J1.42 (Pin_42)
- net PB_{2}: now also J1.44 (Pin_44)
- net PB_{3}: now also J1.46 (Pin_46)
- net PB_{4}: now also J1.48 (Pin_48)
- net PB_{5}: now also J1.50 (Pin_50)
- net PB_{6}: now also J1.52 (Pin_52)
- net PB_{7}: now also J1.54 (Pin_54)
- net PUSBD+: now also J2.A6 (D+), J2.B6 (D+)
- net PUSBD-: now also C8.1, J2.A7 (D-), J2.B7 (D-)
- net USBD-: no longer C8.1
- net VCC: now also D1.2 (A), J1.38 (Pin_38), J1.62 (Pin_62), J1.63 (Pin_63), J2.A4 (VBUS), J2.A9 (VBUS), J2.B4 (VBUS), J2.B9 (VBUS), RN1.1 (R1.1), RN1.2 (R2.1), RN1.3 (R3.1), RN1.4 (R4.1); no longer R7.1
- net ~{ACIACS}: now also J1.57 (Pin_57)
- net ~{IRQ}_{PORT}: now also J1.64 (Pin_64)
- net ~{RAMCS}: now also J1.53 (Pin_53)
- net ~{ROMOE}: now also J1.51 (Pin_51)
- net ~{RST}: now also C10.2, R9.1, SW1.2
- net ~{VIACS}: now also J1.55 (Pin_55)
- net at JP1.2 (B), U1.15 (I/O): now also RN1.8 (R1.2)
- net at R3.1: now also J2.A5 (CC1)
- net at R7.2: now also D1.1 (K); no longer D1.2 (A)
- net at JP2.2 (B), U1.16 (I/O): now also RN1.7 (R2.2)
- net at JP3.2 (B), U1.17 (I/O): now also RN1.6 (R3.2)
- new net: J2.A8 (SBU1), R2.1
- no-connect marks 30 -> 22
Other:
- moved on the sheet: C9, D1, R3, R4, R7, R8

Commit message: More tracing1
Connections:
- net R/~{W}: now also J1.2 (Pin_2)
- no-connect marks 22 -> 21
Changed lines of the file:
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@@
   (no_connect (at 313.69 34.29))
   (no_connect (at 58.42 199.39))
-  (no_connect (at 58.42 196.85))
   (no_connect (at 34.29 35.56))
   (no_connect (at 58.42 207.01))
@@
       (effects (font (size 1.27 1.27)) (justify left) hide)
     )
+  )
+  (global_label "R{slash}~{W}" (shape input) (at 58.42 196.85 0) (fields_autoplaced)
+    (effects (font (size 1.27 1.27)) (justify left))
+    (property "Intersheetrefs" "${INTERSHEET_REFS}" (at 65.4571 196.85 0)
+      (effects (font (size 1.27 1.27)) (justify left) hide)
+    )

Commit message: Finished tracing, corrected INH pull resistor
Parts:
- added R10: 1000, Resistor_SMD:R_1206_3216Metric, symbol Device:R
Connections:
- net GND: now also R10.2
- net INH: now also R10.1
Changed lines of the file:
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@@
   (junction (at 317.5 88.9) (diameter 0) (color 0 0 0 0)
   )
+  (junction (at 71.12 143.51) (diameter 0) (color 0 0 0 0)
+  )
   (junction (at 251.46 176.53) (diameter 0) (color 0 0 0 0)
   )
@@
     (stroke (width 0) (type default))
   )
+  (wire (pts (xy 71.12 143.51) (xy 73.66 143.51))
+    (stroke (width 0) (type default))
+  )
   (wire (pts (xy 251.46 176.53) (xy 259.08 176.53))
     (stroke (width 0) (type default))
@@
     (stroke (width 0) (type default))
   )
+  (wire (pts (xy 67.31 143.51) (xy 71.12 143.51))
+    (stroke (width 0) (type default))
+  )
   (wire (pts (xy 256.54 96.52) (xy 259.08 96.52))
     (stroke (width 0) (type default))
@@
     )
   )
-  (global_label "INH" (shape input) (at 67.31 143.51 0) (fields_autoplaced)
+  (global_label "INH" (shape input) (at 73.66 143.51 0) (fields_autoplaced)
     (effects (font (size 1.27 1.27)) (justify left))
-    (property "Intersheetrefs" "${INTERSHEET_REFS}" (at 73.561 143.51 0)
+    (property "Intersheetrefs" "${INTERSHEET_REFS}" (at 79.911 143.51 0)
       (effects (font (size 1.27 1.27)) (justify left) hide)
     )
@@
     )
   )
+  (symbol (lib_id "power:GND") (at 71.12 151.13 0) (unit 1)
+    (in_bom yes) (on_board yes) (dnp no) (fields_autoplaced)
+    (property "Reference" "#PWR066" (at 71.12 157.48 0)
+      (effects (font (size 1.27 1.27)) hide)
+    )
+    (property "Value" "GND" (at 71.12 156.21 0)
+      (effects (font (size 1.27 1.27)))
+    )
+    (property "Footprint" "" (at 71.12 151.13 0)
+      (effects (font (size 1.27 1.27)) hide)
+    )
+    (property "Datasheet" "" (at 71.12 151.13 0)
+      (effects (font (size 1.27 1.27)) hide)
+    )
+    (pin "1")
+    (instances
+      (project "6502 V1.3"
+        (path "/2462ee6a-a1ab-4fa8-8d76-c1bc8dad46c9"
+          (reference "#PWR066") (unit 1)
+        )
+      )
+    )
+  )
   (symbol (lib_id "power:VCC") (at 220.98 83.82 90) (unit 1)
     (in_bom yes) (on_board yes) (dnp no) (fields_autoplaced)
@@
         )
       )
+    )
+  )
+  (symbol (lib_id "Device:R") (at 71.12 147.32 0) (unit 1)
+    (in_bom yes) (on_board yes) (dnp no) (fields_autoplaced)
+    (property "Reference" "R10" (at 73.66 146.05 0)
+      (effects (font (size 1.27 1.27)) (justify left))
+    )
+    (property "Value" "1000" (at 73.66 148.59 0)
+      (effects (font (size 1.27 1.27)) (justify left))
+    )
+    (property "Footprint" "Resistor_SMD:R_1206_3216Metric" (at 69.342 147.32 90)
+      (effects (font (size 1.27 1.27)) hide)
+    )
+    (property "Datasheet" "~" (at 71.12 147.32 0)
+      (effects (font (size 1.27 1.27)) hide)
+    )
+    (pin "1")
+    (pin "2")
+    (instances
+      (project "6502 V1.3"
+        (path "/2462ee6a-a1ab-4fa8-8d76-c1bc8dad46c9"
+          (reference "R10") (unit 1)
+        )
+      )
