File: KiCad/6502 V1.3-rounded.kicad_pcb (KiCad board)
At the start: 2 copper layers, 152.4 x 76.2 mm, 46 parts, among them J1 USB_C_Receptacle_USB2.0_16P, J2 Conn_02x32_Odd_Even, SW1 SW_DIP_x04, SW2 SW_Push, U1 W65C02SxP, U2 W65C22SxP, U3 W65C51NxP, U4 CY62256-70PC, U5 ATF22V10B-15GM/883, U6 FT230XS, U7 SST39SF040, X1 ACO-1MHz-A, X2 ACO-1.8432MHz-A

Commit message: Fixed 22V10 Socket size, added makefile, created example code
Parts:
- U5: footprint Package_DIP:DIP-24_W10.16mm -> Package_DIP:DIP-24_W7.62mm_Socket
- moved JP3 8.89 mm to (136.4, 68.6)
- moved JP1 8.89 mm to (127.5, 68.6)
- moved G*** 2.40 mm to (148.5, 57.4)
- moved C6 1.94 mm to (130.6, 25.4)
- moved R10 0.06 mm to (113.3, 76.2)
- renumbered C9 to C10, C5 to C4, C4 to C5, C10 to C9, D2 to D1, D1 to D2, R9 to R5, R5 to R9
Connections:
- JP1 pad 1: ~{IRQ}_{PORT} -> ~{IRQ}_{VIA}
- JP1 pad 2: Net-(JP3-B) -> Net-(JP1-B)
- JP3 pad 1: ~{IRQ}_{VIA} -> ~{IRQ}_{PORT}
- JP3 pad 2: Net-(JP1-B) -> Net-(JP3-B)
Routing:
- net ~{ACIACS}: track 124.1 -> 132.8 mm
- net ~{IRQ}_{ACIA}: track 114.1 -> 109.9 mm, vias 0 -> 2
- net ~{VIACS}: track 174.0 -> 177.4 mm
- net Net-(JP1-B): track 28.1 -> 25.3 mm
- net A_{4}: track 208.8 -> 206.1 mm
- net ~{IRQ}_{CPU}: track 165.2 -> 167.7 mm
- net INH: track 62.9 -> 65.3 mm
- net GND: track 443.9 -> 441.5 mm
- net Net-(JP2-B): track 27.3 -> 26.1 mm
- net A_{5}: track 222.4 -> 221.2 mm
- net VCC: track 566.9 -> 565.8 mm
Other:
- board text added: "6502"
- board text added: "6522"
- board text added: "LED_{Rx}"
- board text added: "LED_{Tx}"
- board text added: "PWR"
- board text removed: "65C02"
- board text removed: "65C22"
