File: KiCad/6502 V1.3.kicad_pcb (KiCad board)
At the start: 2 copper layers, 152.4 x 76.2 mm, 45 parts, among them J1 USB_C_Receptacle_USB2.0_16P, J2 Conn_02x32_Odd_Even, SW1 SW_DIP_x04, SW2 SW_Push, U1 W65C02SxP, U2 W65C22SxP, U3 W65C51NxP, U4 CY62256-70PC, U5 ATF22V10B-15GM/883, U6 FT230XS, U7 SST39SF040, X1 ACO-1MHz-A, X2 ACO-1.8432MHz-A

Commit message: Fixed 22V10 Socket size, added makefile, created example code
Parts:
- added G***: LOGO, delorean:unicorn, F.Cu at (148.5, 57.4)
- U5: footprint Package_DIP:DIP-24_W10.16mm -> Package_DIP:DIP-24_W7.62mm_Socket
- moved C6 1.94 mm to (130.6, 25.4)
- renumbered C5 to C4, C4 to C5, JP3 to JP2, JP2 to JP3, R8 to R5, R5 to R6, R6 to R7, R7 to R8
Routing:
- net ~{ACIACS}: track 126.4 -> 135.3 mm
- net ~{IRQ}_{ACIA}: track 117.3 -> 112.5 mm, vias 0 -> 2
- net ~{VIACS}: track 176.5 -> 180.1 mm
- net INH: track 63.9 -> 67.1 mm
- net Net-(JP1-B): track 28.7 -> 25.9 mm
- net A_{4}: track 212.2 -> 209.6 mm
- net ~{IRQ}_{CPU}: track 166.8 -> 169.3 mm
- net GND: track 451.1 -> 448.6 mm
- net VCC: track 575.9 -> 574.3 mm
- net Net-(JP2-B): track 27.7 -> 26.3 mm
- net A_{5}: track 226.2 -> 225.1 mm
Other:
- board text added: "22V10"
- board text added: "39SF040"
- board text added: "4 MHz CLK"
- board text added: "6502"
- board text added: "6502 SBC V1.3 Ethan Thummel 1/22/24"
- board text added: "6522"
- board text added: "6551"
- board text added: "A_{0}"
- board text added: "A_{10}"
- board text added: "A_{11}"
- board text added: "A_{12}"
- board text added: "A_{13}"
- board text added: "A_{14}"
- board text added: "A_{15}"
- board text added: "A_{1}"
- board text added: "A_{2}"
- board text added: "A_{3}"
- board text added: "A_{4}"
- board text added: "A_{5}"
- board text added: "A_{6}"
- board text added: "A_{7}"
- board text added: "A_{8}"
- board text added: "A_{9}"
- board text added: "BANK SELECT"
- board text added: "CA_{1}"
- board text added: "CA_{2}"
- board text added: "CB_{1}"
- board text added: "CB_{2}"
- board text added: "CLK"
- board text added: "D_{0}"
- board text added: "D_{1}"
- board text added: "D_{2}"
- board text added: "D_{3}"
- board text added: "D_{4}"
- board text added: "D_{5}"
- board text added: "D_{6}"
- board text added: "D_{7}"
- board text added: "GND"
- board text added: "HM62256B"
- board text added: "INH"
- board text added: "LED_{Rx}"
- board text added: "LED_{Tx}"
- board text added: "PA_{0}"
- board text added: "PA_{1}"
- board text added: "PA_{2}"
- board text added: "PA_{3}"
- board text added: "PA_{4}"
- board text added: "PA_{5}"
- board text added: "PA_{6}"
- board text added: "PA_{7}"
- board text added: "PB_{0}"
- board text added: "PB_{1}"
- board text added: "PB_{2}"
- board text added: "PB_{3}"
- board text added: "PB_{4}"
- board text added: "PB_{5}"
- board text added: "PB_{6}"
- board text added: "PB_{7}"
- board text added: "PWR"
- board text added: "R/~{W}"
- board text added: "RST"
- board text added: "UART CLK"
- board text added: "VCC"
- board text added: "~{ACIACS}"
- board text added: "~{IRQ}"
- board text added: "~{IRQ}_{ACIA}"
- board text added: "~{IRQ}_{PORT}"
- board text added: "~{IRQ}_{VIA}"
- board text added: "~{RAMCS}"
- board text added: "~{ROMOE}"
- board text added: "~{VIACS}"
- board text added: "コンピューター！"
