File: KiCad/6502 V1.3.kicad_sch (KiCad schematic)
At the start: 41 parts, among them J1 Conn_02x32_Odd_Even, J2 USB_C_Receptacle_USB2.0_16P, SW1 SW_Push, SW2 SW_DIP_x04, U1 ATF22V10B-15GM/883, U2 W65C02SxP, U3 W65C22SxP, U4 W65C51NxP, U5 SST39SF040, U6 FT230XS, U7 CY62256-70PC, X1 ACO-1.8432MHz-A, X2 ACO-1MHz-A

Commit message: Fixed 22V10 Socket size, added makefile, created example code
Parts:
- U1: footprint Package_DIP:DIP-24_W10.16mm -> Package_DIP:DIP-24_W7.62mm_Socket
Changed lines of the file:
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@@
       (effects (font (size 1.524 1.524)))
     )
-    (property "Footprint" "Package_DIP:DIP-24_W10.16mm" (at 26.67 115.57 0)
+    (property "Footprint" "Package_DIP:DIP-24_W7.62mm_Socket" (at 26.67 115.57 0)
       (effects (font (size 1.27 1.27) italic) hide)
     )
